Commit message: Update camera.xacro

File: urdf/camera.xacro (robot description, xacro)
@@ -8,5 +8,5 @@
         <parent link="base_link"/>
         <child link="camera_link"/>
-        <origin xyz="-0.07 0 0.03" rpy="0 -1.57 0"/>
+        <origin xyz="-0.07 0 0.03" rpy="0 0 0"/>
     </joint>
     <link name="camera_link">
