Commit message: Initial commit

File: install/robot_description/share/robot_description/urdf/camera.xacro (robot description, xacro)
@@ -8,5 +8,5 @@
         <parent link="base_link"/>
         <child link="camera_link"/>
-        <origin xyz="-0.07 0 0.03" rpy="0 -1.57 0"/>
+        <origin xyz="0.07 0 0.03" rpy="0 0 0"/>
     </joint>
     <link name="camera_link">
@@ -36,5 +36,5 @@
         <parent link="camera_link"/>
         <child link="camera_link_optical"/>
-        <origin xyz="0 0 0" rpy="3.14 3.14 -1.57"/>
+        <origin xyz="0 0 0" rpy="0 3.14 1.57"/>
     </joint>
     <link name="camera_link_optical">

File: install/robot_description/share/robot_description/urdf/gazebo_control.xacro (robot description, xacro)
@@ -7,5 +7,5 @@
       <left_joint>left_wheel_joint</left_joint>
       <right_joint>right_wheel_joint</right_joint>
-      <wheel_separation>3.14</wheel_separation>
+      <wheel_separation>0.108</wheel_separation>
       <wheel_diameter>0.048</wheel_diameter>
       <!-- Limit -->
@@ -16,5 +16,5 @@
       <frame_id>odom</frame_id>
       <child_frame_id>base_link</child_frame_id>
-      <odom_publisher_frequency>100</odom_publisher_frequency>
+      <odom_publisher_frequency>30</odom_publisher_frequency>
       <tf_topic>/tf</tf_topic>
     </plugin>

File: install/robot_description/share/robot_description/urdf/lidar.xacro (robot description, xacro)
@@ -7,5 +7,5 @@
      <parent link="base_link"/>
      <child link="laser_frame"/>
-     <origin xyz="0 0 0.037" rpy="0 0 0"/>
+     <origin xyz="0 0 0.038" rpy="0 0 0"/>
    </joint>
    <link name="laser_frame">
@@ -36,8 +36,8 @@
    <gazebo reference="laser_frame">
       <sensor name="laser" type="gpu_lidar">
-         <pose> 0 0 0 0 0 0 </pose>
+         <pose> 0 0 0.2 0 0 0 </pose>
          <always_on>true</always_on>
          <visualize>true</visualize>
-         <update_rate>15</update_rate>
+         <update_rate>10</update_rate>
          <topic>/scan</topic>
          <gz_frame_id>laser_frame</gz_frame_id>
@@ -52,5 +52,5 @@
             <range>
                <min>0.1</min>
-               <max>20</max>
+               <max>8</max>
             </range>
          </lidar>

File: install/robot_description/share/robot_description/urdf/robot_core.xacro (robot description, xacro)
@@ -61,5 +61,5 @@
         <parent link="base_link"/>
         <child link="caster_support"/>
-        <origin xyz="-0.065 0 -0.01" rpy="0 0 0"/>
+        <origin xyz="-0.085 0 -0.01" rpy="0 0 0"/>
     </joint>
     <link name="caster_support">
@@ -68,5 +68,5 @@
                 <box size="0.02 0.02 0.04"/>
             </geometry>
-            <origin xyz="-0.01 0 0" rpy="0 0 0"/>
+            <origin xyz="0.01 0 0" rpy="0 0 0"/>
             <material name="grey"/>
         </visual>
@@ -75,9 +75,9 @@
                 <box size="0.02 0.02 0.04"/>
             </geometry>
-            <origin xyz="-0.01 0 0" rpy="0 0 0"/>
+            <origin xyz="0.01 0 0" rpy="0 0 0"/>
         </collision>
         <inertial>
             <mass value="0.25" />
-            <origin xyz="-0.01 0 0" rpy="0 0 0"/>
+            <origin xyz="0.01 0 0" rpy="0 0 0"/>
             <inertia ixx="1.66666666666667e-5" ixy="0.0" ixz="0.0"
                     iyy="2.66666666666667e-5" iyz="0.0"
@@ -88,5 +88,5 @@
         <visual>
             <geometry>
-                <cylinder length="0.005" radius="0.02"/>
+                <cylinder length="0.005" radius="0.01"/>
             </geometry>
             <origin rpy="-1.5708 0 0"/>
@@ -95,14 +95,15 @@
         <collision>
             <geometry>
-                <cylinder length="0.005" radius="0.02"/>
+                <cylinder length="0.005" radius="0.01"/>
             </geometry>
             <origin rpy="-1.5708 0 0"/>
         </collision>
         <inertial>
-            <mass value="0.1" />
+            <mass value="0.01" />
             <origin rpy="-1.5708 0 0"/>
-            <inertia ixx="1.02083333333333e-5" ixy="0.0" ixz="0.0"
-                    iyy="1.02083333333333e-5" iyz="0.0"
-                    izz="2e-5" />
+              <inertia
+                   ixx="0.0000005" ixy="0.0" ixz="0.0"
+                   iyy="0.000000270833" iyz="0.0"
+                   izz="0.000000270833"/>
         </inertial>
     </link>
@@ -111,5 +112,5 @@
         <parent link="caster_support"/>
         <child link="caster_wheel"/>
-        <origin xyz="-0.02 0 -0.02" rpy="0 0 0" />
+        <origin xyz="-0.006 0 -0.02" rpy="0 0 0" />
         <dynamics damping="0.3" friction="0.0"/>
     </joint>
@@ -140,5 +141,5 @@
         <parent link="base_link"/>
         <child link="right_wheel"/>
-        <origin xyz="0 0.054 -0.021"/>
+        <origin xyz="0.03 -0.054 -0.021"/>
         <dynamics damping="0.1" friction="0.0"/>
     </joint>
@@ -169,5 +170,5 @@
         <parent link="base_link"/>
         <child link="left_wheel"/>
-        <origin xyz="0 -0.054 -0.021"/>
+        <origin xyz="0.03 0.054 -0.021"/>
         <dynamics damping="0.1" friction="0.0"/>
   </joint>
